File: thruster-pcb/thruster-pcb.kicad_sch (KiCad schematic)
At the start: 0 parts

Commit message: tmc5160-usb -> thruster-pcb
Other:
- title: tmc5160-usb -> thruster-pcb
Changed lines of the file:
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@@
   (paper "A4")
   (title_block
-    (title "tmc5160-usb")
+    (title "thruster-pcb")
     (date "2024-05-10")
     (rev "1.0")
@@
     )
     (instances
-      (project "tmc5160-usb"
+      (project "thruster-pcb"
         (path "/df2b2e89-e055-4140-95de-f1df723db034" (page "4"))
       )
@@
     )
     (instances
-      (project "tmc5160-usb"
+      (project "thruster-pcb"
         (path "/df2b2e89-e055-4140-95de-f1df723db034" (page "2"))
       )
@@
     )
     (instances
-      (project "tmc5160-usb"
+      (project "thruster-pcb"
         (path "/df2b2e89-e055-4140-95de-f1df723db034" (page "13"))
       )
@@
     )
     (instances
-      (project "tmc5160-usb"
+      (project "thruster-pcb"
         (path "/df2b2e89-e055-4140-95de-f1df723db034" (page "3"))
       )

Commit message: Add reference files
Other:
- removed sheet tmc5160
- company: Howard Hughes Medical Institute -> Mechatronic Magic
Changed lines of the file:
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@@
   (title_block
     (title "thruster-pcb")
-    (date "2024-05-10")
+    (date "2025-01-04")
     (rev "1.0")
-    (company "Howard Hughes Medical Institute")
+    (company "Mechatronic Magic")
   )
   (wire (pts (xy 130.81 102.87) (xy 128.27 102.87))
-    (stroke (width 0) (type default))
-  )
-  (wire (pts (xy 130.81 128.27) (xy 128.27 128.27))
     (stroke (width 0) (type default))
   )
@@
     (stroke (width 0) (type default))
   )
-  (wire (pts (xy 128.27 118.11) (xy 130.81 118.11))
-    (stroke (width 0) (type default))
-  )
-  (wire (pts (xy 130.81 130.81) (xy 128.27 130.81))
-    (stroke (width 0) (type default))
-  )
   (wire (pts (xy 154.94 67.31) (xy 152.4 67.31))
-    (stroke (width 0) (type default))
-  )
-  (wire (pts (xy 130.81 125.73) (xy 128.27 125.73))
-    (stroke (width 0) (type default))
-  )
-  (wire (pts (xy 152.4 130.81) (xy 154.94 130.81))
     (stroke (width 0) (type default))
   )
@@
   )
   (wire (pts (xy 128.27 55.88) (xy 130.81 55.88))
-    (stroke (width 0) (type default))
-  )
-  (wire (pts (xy 128.27 115.57) (xy 130.81 115.57))
-    (stroke (width 0) (type default))
-  )
-  (wire (pts (xy 152.4 128.27) (xy 154.94 128.27))
-    (stroke (width 0) (type default))
-  )
-  (wire (pts (xy 152.4 125.73) (xy 154.94 125.73))
-    (stroke (width 0) (type default))
-  )
-  (wire (pts (xy 128.27 120.65) (xy 130.81 120.65))
     (stroke (width 0) (type default))
   )
@@
     (effects (font (size 1.27 1.27)) (justify left bottom))
   )
-  (label "DIAG1" (at 154.94 130.81 0) (fields_autoplaced)
-    (effects (font (size 1.27 1.27)) (justify left bottom))
-  )
   (label "VIO" (at 154.94 72.39 0) (fields_autoplaced)
     (effects (font (size 1.27 1.27)) (justify left bottom))
@@
   (label "+5V" (at 154.94 69.85 0) (fields_autoplaced)
     (effects (font (size 1.27 1.27)) (justify left bottom))
-  )
-  (label "COPI" (at 128.27 130.81 180) (fields_autoplaced)
-    (effects (font (size 1.27 1.27)) (justify right bottom))
   )
   (label "ENABLE_VIO" (at 154.94 100.33 0) (fields_autoplaced)
@@
     (effects (font (size 1.27 1.27)) (justify right bottom))
   )
-  (label "VIO" (at 128.27 118.11 180) (fields_autoplaced)
-    (effects (font (size 1.27 1.27)) (justify right bottom))
-  )
-  (label "VM" (at 128.27 115.57 180) (fields_autoplaced)
-    (effects (font (size 1.27 1.27)) (justify right bottom))
-  )
   (label "SCK" (at 154.94 95.25 0) (fields_autoplaced)
-    (effects (font (size 1.27 1.27)) (justify left bottom))
-  )
-  (label "DIAG0" (at 154.94 128.27 0) (fields_autoplaced)
     (effects (font (size 1.27 1.27)) (justify left bottom))
   )
@@
     (effects (font (size 1.27 1.27)) (justify left bottom))
   )
-  (label "GND" (at 128.27 120.65 180) (fields_autoplaced)
-    (effects (font (size 1.27 1.27)) (justify right bottom))
-  )
-  (label "CIPO" (at 154.94 125.73 0) (fields_autoplaced)
-    (effects (font (size 1.27 1.27)) (justify left bottom))
-  )
   (label "ENABLE_VIO" (at 128.27 72.39 180) (fields_autoplaced)
-    (effects (font (size 1.27 1.27)) (justify right bottom))
-  )
-  (label "SCK" (at 128.27 128.27 180) (fields_autoplaced)
     (effects (font (size 1.27 1.27)) (justify right bottom))
   )
   (label "~{CS}" (at 154.94 92.71 0) (fields_autoplaced)
     (effects (font (size 1.27 1.27)) (justify left bottom))
-  )
-  (label "~{CS}" (at 128.27 125.73 180) (fields_autoplaced)
-    (effects (font (size 1.27 1.27)) (justify right bottom))
   )
   (label "ENABLE_FAN" (at 128.27 74.93 180) (fields_autoplaced)
@@
     (effects (font (size 1.27 1.27)) (justify right bottom))
   )
-  (sheet (at 130.81 113.03) (size 21.59 20.32) (fields_autoplaced)
-    (stroke (width 0.1524) (type solid))
-    (fill (color 0 0 0 0.0000))
-    (property "Sheetname" "tmc5160" (at 130.81 112.3184 0)
-      (effects (font (size 1.27 1.27)) (justify left bottom))
-    )
-    (property "Sheetfile" "tmc5160.kicad_sch" (at 130.81 133.9346 0)
-      (effects (font (size 1.27 1.27)) (justify left top))
-    )
-    (pin "VM" passive (at 130.81 115.57 180)
-      (effects (font (size 1.27 1.27)) (justify left))
-    )
-    (pin "VIO" passive (at 130.81 118.11 180)
-      (effects (font (size 1.27 1.27)) (justify left))
-    )
-    (pin "GND" passive (at 130.81 120.65 180)
-      (effects (font (size 1.27 1.27)) (justify left))
-    )
-    (pin "~{CS}" input (at 130.81 125.73 180)
-      (effects (font (size 1.27 1.27)) (justify left))
-    )
-    (pin "SCK" input (at 130.81 128.27 180)
-      (effects (font (size 1.27 1.27)) (justify left))
-    )
-    (pin "DIAG0" output (at 152.4 128.27 0)
-      (effects (font (size 1.27 1.27)) (justify right))
-    )
-    (pin "DIAG1" output (at 152.4 130.81 0)
-      (effects (font (size 1.27 1.27)) (justify right))
-    )
-    (pin "CIPO" output (at 152.4 125.73 0)
-      (effects (font (size 1.27 1.27)) (justify right))
-    )
-    (pin "COPI" input (at 130.81 130.81 180)
-      (effects (font (size 1.27 1.27)) (justify left))
-    )
-    (instances
-      (project "thruster-pcb"
-        (path "/df2b2e89-e055-4140-95de-f1df723db034" (page "4"))
-      )
-    )
-  )
   (sheet (at 130.81 53.34) (size 21.59 5.08) (fields_autoplaced)

Commit message: Add parts to schematic
Parts:
- added C1, C11, C12, C15, C17, C18, C19, C7, C8: 100n, pkl_dipol:C_0402, symbol pkl_device:pkl_C_Small
- added C10: 10u, pkl_dipol:C_0603, symbol pkl_device:pkl_C
- added C13, C16: 10n, pkl_dipol:C_0402, symbol pkl_device:pkl_C_Small
- added C14, C2, C9: 1u, pkl_dipol:C_0402, symbol pkl_device:pkl_C_Small
- added C3, C4, C5, C6: 4u7, pkl_dipol:C_0603, symbol pkl_device:pkl_C
- added D1: BLU, pkl_dipol:D_0603, symbol pkl_device:pkl_LED_Small
- added D2: RED, pkl_dipol:D_0603, symbol pkl_device:pkl_LED_Small
- added D3: GRN, pkl_dipol:D_0603, symbol pkl_device:pkl_LED_Small
- added D4: FM-B2020RGBA-HG, pkl_led:LED_TRI_2020, symbol pkl_device:pkl_LED_RBAG
- added J1: USB_C, pkl_connectors:USB_C_Receptacle_HRO_TYPE-C-31-M-12, symbol Connector:USB_C_Receptacle_USB2.0
- added JP1: VIN-VBUS, pkl_jumpers:J_NC_0603_40, symbol pkl_misc:pkl_jumper_nc
- added JP2: RAM_CS-LEDG, pkl_jumpers:J_NC_0402_15, symbol pkl_misc:pkl_jumper_nc
- added JP3: Flash_CS-SPI_CS, pkl_jumpers:J_NC_0402_15, symbol pkl_misc:pkl_jumper_nc
- added JP4: VccIO2, pkl_jumpers:J_NC_0603_30, symbol pkl_misc:pkl_jumper_nc
- added JP5: Vpp2v5, pkl_jumpers:J_NC_0402_30, symbol pkl_misc:pkl_jumper_nc
- added JP6: VccIO0, pkl_jumpers:J_NC_0603_30, symbol pkl_misc:pkl_jumper_nc
- added LOGO1: 1BitSquared, pkl_logos:1b2_Logo_SilkS_2mm, symbol pkl_logos:1BitSquared
- added P1, P2, P3, P4: UP, pkl_pads:PAD_SMD_1x2.65_ROUNDED, symbol pkl_misc:PAD_SMD
- added P10: IO2, pkl_pads:PAD_SMD_R_1x1, symbol Connector_Generic:Conn_01x01
- added P11, P12, P20: GND, pkl_pin_headers:Pin_Header_Straight_Round_1x01_Castellated, symbol Connector_Generic:Conn_01x01
- added P13: 23, pkl_pin_headers:Pin_Header_Straight_Round_1x01_Castellated, symbol Connector_Generic:Conn_01x01
- added P14: 0, pkl_pin_headers:Pin_Header_Straight_Round_1x01_Castellated, symbol Connector_Generic:Conn_01x01
- added P15: 1, pkl_pin_headers:Pin_Header_Straight_Round_1x01_Castellated, symbol Connector_Generic:Conn_01x01
- added P16: 2, pkl_pin_headers:Pin_Header_Straight_Round_1x01_Castellated, symbol Connector_Generic:Conn_01x01
- added P17: 3, pkl_pin_headers:Pin_Header_Straight_Round_1x01_Castellated, symbol Connector_Generic:Conn_01x01
- added P18: 4, pkl_pin_headers:Pin_Header_Straight_Round_1x01_Castellated, symbol Connector_Generic:Conn_01x01
- added P19: 5, pkl_pin_headers:Pin_Header_Straight_Round_1x01_Castellated, symbol Connector_Generic:Conn_01x01
- added P21, P22: 3V3, pkl_pin_headers:Pin_Header_Straight_Round_1x01_Castellated, symbol Connector_Generic:Conn_01x01
- added P23: VIN, pkl_pin_headers:Pin_Header_Straight_Round_1x01_Castellated, symbol Connector_Generic:Conn_01x01
- added P24: 13, pkl_pin_headers:Pin_Header_Straight_Round_1x01_Castellated, symbol Connector_Generic:Conn_01x01
- added P25: 14, pkl_pin_headers:Pin_Header_Straight_Round_1x01_Castellated, symbol Connector_Generic:Conn_01x01
- added P26: 15, pkl_pin_headers:Pin_Header_Straight_Round_1x01_Castellated, symbol Connector_Generic:Conn_01x01
- added P27: 16, pkl_pin_headers:Pin_Header_Straight_Round_1x01_Castellated, symbol Connector_Generic:Conn_01x01
- added P28: 17, pkl_pin_headers:Pin_Header_Straight_Round_1x01_Castellated, symbol Connector_Generic:Conn_01x01
- added P29: 18, pkl_pin_headers:Pin_Header_Straight_Round_1x01_Castellated, symbol Connector_Generic:Conn_01x01
- added P30: 19, pkl_pin_headers:Pin_Header_Straight_Round_1x01_Castellated, symbol Connector_Generic:Conn_01x01
- added P31: 20, pkl_pin_headers:Pin_Header_Straight_Round_1x01_Castellated, symbol Connector_Generic:Conn_01x01
- added P32: 21, pkl_pin_headers:Pin_Header_Straight_Round_1x01_Castellated, symbol Connector_Generic:Conn_01x01
- added P33: 22, pkl_pin_headers:Pin_Header_Straight_Round_1x01_Castellated, symbol Connector_Generic:Conn_01x01
- added P34: 6, pkl_pin_headers:Pin_Header_Straight_Round_1x01_Castellated, symbol Connector_Generic:Conn_01x01
- added P35: 7, pkl_pin_headers:Pin_Header_Straight_Round_1x01_Castellated, symbol Connector_Generic:Conn_01x01
- added P36: 8, pkl_pin_headers:Pin_Header_Straight_Round_1x01_Castellated, symbol Connector_Generic:Conn_01x01
- added P37: 9, pkl_pin_headers:Pin_Header_Straight_Round_1x01_Castellated, symbol Connector_Generic:Conn_01x01
- added P38: 10, pkl_pin_headers:Pin_Header_Straight_Round_1x01_Castellated, symbol Connector_Generic:Conn_01x01
- added P39: 11, pkl_pin_headers:Pin_Header_Straight_Round_1x01_Castellated, symbol Connector_Generic:Conn_01x01
- added P40: 12, pkl_pin_headers:Pin_Header_Straight_Round_1x01_Castellated, symbol Connector_Generic:Conn_01x01
- added P41: CDONE, pkl_pin_headers:Pin_Header_Straight_Round_1x01_Castellated, symbol Connector_Generic:Conn_01x01
- added P42: CRESET, pkl_pin_headers:Pin_Header_Straight_Round_1x01_Castellated, symbol Connector_Generic:Conn_01x01
- added P5: CS, pkl_pin_headers:Pin_Header_Straight_Round_1x01, symbol Connector_Generic:Conn_01x01
- added P6: SCK, pkl_pin_headers:Pin_Header_Straight_Round_1x01, symbol Connector_Generic:Conn_01x01
- added P7: CIPO, pkl_pin_headers:Pin_Header_Straight_Round_1x01, symbol Connector_Generic:Conn_01x01
- added P8: COPI, pkl_pin_headers:Pin_Header_Straight_Round_1x01, symbol Connector_Generic:Conn_01x01
- added P9: IO3, pkl_pads:PAD_SMD_R_1x1, symbol Connector_Generic:Conn_01x01
- added R1: 1M, pkl_dipol:R_0402, symbol pkl_device:pkl_R_Small
- added R10, R9: 22E, pkl_dipol:R_0402, symbol pkl_device:pkl_R_Small
- added R11, R12, R13: 2k2, pkl_dipol:R_0402, symbol pkl_device:pkl_R_Small
- added R14: 100E, pkl_dipol:R_0402, symbol pkl_device:pkl_R_Small
- added R2, R6, R8: 10k, pkl_dipol:R_0402, symbol pkl_device:pkl_R_Small
- added R3, R4: 5k1, pkl_dipol:R_0402, symbol pkl_device:pkl_R_Small
- added R5: 10k, pkl_dipol:R_Array_Convex_4x0402, symbol pkl_device:pkl_R4_Small
- added R7: 1k5, pkl_dipol:R_0402, symbol pkl_device:pkl_R_Small
- added SW1: TACT, pkl_buttons_switches:SW_SPST_3x4x2.5, symbol pkl_misc:TACT
- added TP1: CC1, pkl_misc:TestPoint_Pad_D0.75mm, symbol Connector:TestPoint_Small
- added TP2: CC2, pkl_misc:TestPoint_Pad_D0.75mm, symbol Connector:TestPoint_Small
- added TP3: SBU1, pkl_misc:TestPoint_Pad_D0.75mm, symbol Connector:TestPoint_Small
- added TP4: SBU2, pkl_misc:TestPoint_Pad_D0.75mm, symbol Connector:TestPoint_Small
- added U1: LY68L6400, Package_SO:SOIC-8_3.9x4.9mm_P1.27mm, symbol pkl_memory:VTI7064
- added U2: W25Q128JVxxM, Package_SON:WSON-8-1EP_6x5mm_P1.27mm_EP3.4x4.3mm, symbol pkl_memory:W25Q
- added U3: TLV75533PDRV, Package_SON:WSON-6-1EP_2x2mm_P0.65mm_EP1x1.6mm, symbol Regulator_Linear:TLV75533PDRV
- added U4: USBLC6-2, pkl_housings_sot:SOT-666, symbol pkl_misc:USBLC6-2
- added U5: TLV73312PDRV, Package_SON:WSON-6-1EP_2x2mm_P0.65mm_EP1x1.6mm, symbol Regulator_Linear:TLV75512PDRV
- added U6: ICE40UP5K-SG48, pkl_housings_dfn_qfn:QFN-48-1EP_7x7mm_Pitch0.5mm, symbol pkl_lattice:ICE40UP5K-SG48
- added X1: 12MHz, pkl_misc:Oscillator_SMD_SCTF_S2DXX-4Pin_2.5x2.0mm, symbol Oscillator:ASE-xxxMHz
Connections:
- net GND: now also C1.2, C10.2, C11.2, C12.2, C13.2, C14.2, C15.2, C16.2, C17.2, C18.2, C19.2, C2.2, C3.2, C4.2, C5.2, C6.2, C7.2, C8.2, C9.2, D1.C, J1.A1 (GND), J1.A12 (GND), J1.B1 (GND), J1.B12 (GND), P11.1 (Pin_1), P12.1 (Pin_1), P20.1 (Pin_1), P4.1 (PAD), R1.1, R3.1, R4.1, SW1.1, U1.4 (GND), U2.4 (GND), U3.3 (GND), U3.7 (GND), U4.2 (GND), U5.3 (GND), U5.7 (GND), U6.49 (PAD/GND), X1.2 (GND)
- new net: D2.A, R11.1
- new net: D3.A, R12.1
- new net +1V2: C11.1, C13.1, C14.1, C15.1, C16.1, C6.1, C9.1, R14.2, U5.1 (OUT), U6.30 (VCC), U6.5 (VCC)
- new net +3V3: C1.1, C19.1, C4.1, C7.1, D4.3 (A), JP4.2, JP5.1, JP6.2, P21.1 (Pin_1), P22.1 (Pin_1), R11.2, R12.2, R13.2, R5.1, R5.3, R5.6, R5.8, R8.1, U1.8 (VCC), U2.8 (VCC), U3.1 (OUT), U6.22 (SPI_VCCIO1), X1.4 (Vdd)
- new net 3V3_EN: C2.1, R2.2, U3.4 (EN)
- new net CC1: J1.A5 (CC1), R3.2, TP1.1
- new net CC2: J1.B5 (CC2), R4.2, TP2.1
- new net CDONE: D1.A, P41.1 (Pin_1), R13.1, U6.7 (CDONE)
- new net CLK: U6.35 (IOT_46B_G0), X1.3 (OUT)
- new net CLK_EN: R8.2, X1.1 (EN)
- new net FLASH_~{CS}: JP3.1, R5.4, U2.1 (~{CS})
- new net IOB_0a: P13.1 (Pin_1), U6.46 (IOB_0A)
- new net IOB_13b-~{LEDG}: D3.C, JP2.2, U6.6 (IOB_13B)
- new net IOB_16a: P34.1 (Pin_1), U6.9 (IOB_16A)
- new net IOB_18a: P35.1 (Pin_1), U6.10 (IOB_18A)
- new net IOB_20a: P36.1 (Pin_1), U6.11 (IOB_20A)
- new net IOB_22a: P37.1 (Pin_1), U6.12 (IOB_22A)
- new net IOB_23b: P38.1 (Pin_1), U6.21 (IOB_23B)
- new net IOB_24a: P39.1 (Pin_1), U6.13 (IOB_24A)
- new net IOB_25b_G3: P40.1 (Pin_1), U6.20 (IOB_25B_G3)
- new net IOB_2a: P14.1 (Pin_1), U6.47 (IOB_2A)
- new net IOB_3b_G6: P15.1 (Pin_1), U6.44 (IOB_3B_G6)
- new net IOB_4a: P16.1 (Pin_1), U6.48 (IOB_4A)
- new net IOB_5b: P17.1 (Pin_1), U6.45 (IOB_5B)
- new net IOB_8a: P18.1 (Pin_1), U6.4 (IOB_8A)
- new net IOB_9b: P19.1 (Pin_1), U6.3 (IOB_9B)
- new net IOT_36b-~{LEDR}: D2.C, P24.1 (Pin_1), U6.25 (IOT_36B)
- new net IOT_37a: P25.1 (Pin_1), U6.23 (IOT_37A)
- new net IOT_38b: P26.1 (Pin_1), U6.27 (IOT_38B)
- new net IOT_39a: P27.1 (Pin_1), U6.26 (IOT_39A)
- new net IOT_41a: P28.1 (Pin_1), U6.28 (IOT_41A)
- new net IOT_42b: P29.1 (Pin_1), U6.31 (IOT_42B)
- new net IOT_43a: P30.1 (Pin_1), U6.32 (IOT_43A)
- new net IOT_44b: P31.1 (Pin_1), U6.34 (IOT_44B)
- new net IOT_48b: P32.1 (Pin_1), U6.36 (IOT_48B)
- new net IOT_49a: P33.1 (Pin_1), U6.43 (IOT_49A)
- new net RAM_~{CS}: JP2.1, R5.7, U1.1 (~{CE})
- new net SBU1: J1.A8 (SBU1), TP3.1
- new net SBU2: J1.B8 (SBU2), TP4.1
- new net SHIELD: J1.S1 (SHIELD), R1.2
- new net SPI_CIPO-IO1: P7.1 (Pin_1), U1.2 (SO/SIO1), U2.2 (DO/IO1), U6.17 (IOB_33b_SPI_SI)
- new net SPI_COPI-IO0: P8.1 (Pin_1), U1.5 (SI/SIO0), U2.5 (DI/IO0), U6.14 (IOB_32a_SPI_SO)
- new net SPI_SCK: P6.1 (Pin_1), R5.2, U1.6 (SCLK), U2.6 (CLK), U6.15 (IOB_34a_SPI_SCK)
- new net SPI_~{CS}: JP3.2, P5.1 (Pin_1), U6.16 (IOB_35b_SPI_CSN)
- new net SPI_~{HLD}-IO3: P9.1 (Pin_1), U1.7 (SIO3), U2.7 (~{HLD}/~{RST}/IO3), U6.19 (IOB_29B)
- new net SPI_~{WP}-IO2: P10.1 (Pin_1), U1.3 (SIO2), U2.3 (~{WP}/IO2), U6.18 (IOB_31B)
- new net USB_DET: R7.1, U6.37 (IOT_45A_G1)
- new net USB_N: R9.1, U6.38 (IOT_50B)
- new net USB_P: R10.1, U6.42 (IOT_51A)
- new net VBUS: J1.A4 (VBUS), J1.A9 (VBUS), J1.B4 (VBUS), J1.B9 (VBUS), JP1.1, P1.1 (PAD), U4.5 (VBUS)
- new net VCCIO_0: C18.1, JP6.1, U6.33 (VCCIO_0)
- new net VCCIO_2: C8.1, JP4.1, R6.2, U6.1 (VCCIO_2)
- new net VCCPLL: C10.1, C12.1, R14.1, U6.29 (VCCPLL)
- new net VIN: C3.1, C5.1, JP1.2, P23.1 (Pin_1), R2.1, U3.6 (IN), U5.4 (EN), U5.6 (IN)
- new net VPP_2V5: C17.1, JP5.2, U6.24 (VPP_2V5)
- new net iD+: R10.2, R7.2, U4.4 (IO2)
- new net iD-: R9.2, U4.6 (IO1)
- new net xD+: J1.A6 (D+), J1.B6 (D+), P3.1 (PAD), U4.3 (IO2)
- new net xD-: J1.A7 (D-), J1.B7 (D-), P2.1 (PAD), U4.1 (IO1)
- new net ~{BTN}: R6.1, SW1.2, U6.2 (IOB_6A)
- new net ~{CRESET}: P42.1 (Pin_1), R5.5, U6.8 (CRESET_B)
- new net ~{RGB0}: D4.1 (RK), U6.39 (RGB0)
- new net ~{RGB1}: D4.4 (GK), U6.40 (RGB1)
- new net ~{RGB2}: D4.2 (BK), U6.41 (RGB2)
Other:
- note added: "+"
- note added: "-"
- note added: "128M Flash"
- note added: "1V2 VReg"
- note added: "3V3 VReg"
- note added: "64M PSRAM"
- note added: "Button"
- note added: "Chip Select"
- note added: "Clock"
- note added: "DPair"
- note added: "Enable Delay ~1 millisecond Should enable after 1V2 rail"
- note added: "FPGA"
- note added: "Flash/RAM"
- note added: "Hold"
- note added: "JP3: Cut jumper when only programming iCE Connect jumper for programming Flash and for normal operation"
- note added: "LEDs"
- note added: "Main In Secondary Out"
- note added: "Main Out Secondary In"
- note added: "Power Pins"
- note added: "QSPI/Programming"
- note added: "Serial Clock"
- note added: "USB"
- note added: "Using same values as STM32F1 spec"
- note added: "Write Protect"
- note added: "or less"

Commit message: Use PCA9685 and nRF52
Parts:
- removed C1, C11, C12, C15, C17, C18, C19, C7, C8: 100n, pkl_dipol:C_0402, symbol pkl_device:pkl_C_Small
- removed C10: 10u, pkl_dipol:C_0603, symbol pkl_device:pkl_C
- removed C13, C16: 10n, pkl_dipol:C_0402, symbol pkl_device:pkl_C_Small
- removed C14, C2, C9: 1u, pkl_dipol:C_0402, symbol pkl_device:pkl_C_Small
- removed C3, C4, C5, C6: 4u7, pkl_dipol:C_0603, symbol pkl_device:pkl_C
- removed D1: BLU, pkl_dipol:D_0603, symbol pkl_device:pkl_LED_Small
- removed D2: RED, pkl_dipol:D_0603, symbol pkl_device:pkl_LED_Small
- removed D3: GRN, pkl_dipol:D_0603, symbol pkl_device:pkl_LED_Small
- removed D4: FM-B2020RGBA-HG, pkl_led:LED_TRI_2020, symbol pkl_device:pkl_LED_RBAG
- removed J1: USB_C, pkl_connectors:USB_C_Receptacle_HRO_TYPE-C-31-M-12, symbol Connector:USB_C_Receptacle_USB2.0
- removed JP1: VIN-VBUS, pkl_jumpers:J_NC_0603_40, symbol pkl_misc:pkl_jumper_nc
- removed JP2: RAM_CS-LEDG, pkl_jumpers:J_NC_0402_15, symbol pkl_misc:pkl_jumper_nc
- removed JP3: Flash_CS-SPI_CS, pkl_jumpers:J_NC_0402_15, symbol pkl_misc:pkl_jumper_nc
- removed JP4: VccIO2, pkl_jumpers:J_NC_0603_30, symbol pkl_misc:pkl_jumper_nc
- removed JP5: Vpp2v5, pkl_jumpers:J_NC_0402_30, symbol pkl_misc:pkl_jumper_nc
- removed JP6: VccIO0, pkl_jumpers:J_NC_0603_30, symbol pkl_misc:pkl_jumper_nc
- removed LOGO1: 1BitSquared, pkl_logos:1b2_Logo_SilkS_2mm, symbol pkl_logos:1BitSquared
- removed P1, P2, P3, P4: UP, pkl_pads:PAD_SMD_1x2.65_ROUNDED, symbol pkl_misc:PAD_SMD
- removed P10: IO2, pkl_pads:PAD_SMD_R_1x1, symbol Connector_Generic:Conn_01x01
- removed P11, P12, P20: GND, pkl_pin_headers:Pin_Header_Straight_Round_1x01_Castellated, symbol Connector_Generic:Conn_01x01
- removed P13: 23, pkl_pin_headers:Pin_Header_Straight_Round_1x01_Castellated, symbol Connector_Generic:Conn_01x01
- removed P14: 0, pkl_pin_headers:Pin_Header_Straight_Round_1x01_Castellated, symbol Connector_Generic:Conn_01x01
- removed P15: 1, pkl_pin_headers:Pin_Header_Straight_Round_1x01_Castellated, symbol Connector_Generic:Conn_01x01
- removed P16: 2, pkl_pin_headers:Pin_Header_Straight_Round_1x01_Castellated, symbol Connector_Generic:Conn_01x01
- removed P17: 3, pkl_pin_headers:Pin_Header_Straight_Round_1x01_Castellated, symbol Connector_Generic:Conn_01x01
- removed P18: 4, pkl_pin_headers:Pin_Header_Straight_Round_1x01_Castellated, symbol Connector_Generic:Conn_01x01
- removed P19: 5, pkl_pin_headers:Pin_Header_Straight_Round_1x01_Castellated, symbol Connector_Generic:Conn_01x01
- removed P21, P22: 3V3, pkl_pin_headers:Pin_Header_Straight_Round_1x01_Castellated, symbol Connector_Generic:Conn_01x01
- removed P23: VIN, pkl_pin_headers:Pin_Header_Straight_Round_1x01_Castellated, symbol Connector_Generic:Conn_01x01
- removed P24: 13, pkl_pin_headers:Pin_Header_Straight_Round_1x01_Castellated, symbol Connector_Generic:Conn_01x01
- removed P25: 14, pkl_pin_headers:Pin_Header_Straight_Round_1x01_Castellated, symbol Connector_Generic:Conn_01x01
- removed P26: 15, pkl_pin_headers:Pin_Header_Straight_Round_1x01_Castellated, symbol Connector_Generic:Conn_01x01
- removed P27: 16, pkl_pin_headers:Pin_Header_Straight_Round_1x01_Castellated, symbol Connector_Generic:Conn_01x01
- removed P28: 17, pkl_pin_headers:Pin_Header_Straight_Round_1x01_Castellated, symbol Connector_Generic:Conn_01x01
- removed P29: 18, pkl_pin_headers:Pin_Header_Straight_Round_1x01_Castellated, symbol Connector_Generic:Conn_01x01
- removed P30: 19, pkl_pin_headers:Pin_Header_Straight_Round_1x01_Castellated, symbol Connector_Generic:Conn_01x01
- removed P31: 20, pkl_pin_headers:Pin_Header_Straight_Round_1x01_Castellated, symbol Connector_Generic:Conn_01x01
- removed P32: 21, pkl_pin_headers:Pin_Header_Straight_Round_1x01_Castellated, symbol Connector_Generic:Conn_01x01
- removed P33: 22, pkl_pin_headers:Pin_Header_Straight_Round_1x01_Castellated, symbol Connector_Generic:Conn_01x01
- removed P34: 6, pkl_pin_headers:Pin_Header_Straight_Round_1x01_Castellated, symbol Connector_Generic:Conn_01x01
- removed P35: 7, pkl_pin_headers:Pin_Header_Straight_Round_1x01_Castellated, symbol Connector_Generic:Conn_01x01
- removed P36: 8, pkl_pin_headers:Pin_Header_Straight_Round_1x01_Castellated, symbol Connector_Generic:Conn_01x01
- removed P37: 9, pkl_pin_headers:Pin_Header_Straight_Round_1x01_Castellated, symbol Connector_Generic:Conn_01x01
- removed P38: 10, pkl_pin_headers:Pin_Header_Straight_Round_1x01_Castellated, symbol Connector_Generic:Conn_01x01
- removed P39: 11, pkl_pin_headers:Pin_Header_Straight_Round_1x01_Castellated, symbol Connector_Generic:Conn_01x01
- removed P40: 12, pkl_pin_headers:Pin_Header_Straight_Round_1x01_Castellated, symbol Connector_Generic:Conn_01x01
- removed P41: CDONE, pkl_pin_headers:Pin_Header_Straight_Round_1x01_Castellated, symbol Connector_Generic:Conn_01x01
- removed P42: CRESET, pkl_pin_headers:Pin_Header_Straight_Round_1x01_Castellated, symbol Connector_Generic:Conn_01x01
- removed P5: CS, pkl_pin_headers:Pin_Header_Straight_Round_1x01, symbol Connector_Generic:Conn_01x01
- removed P6: SCK, pkl_pin_headers:Pin_Header_Straight_Round_1x01, symbol Connector_Generic:Conn_01x01
- removed P7: CIPO, pkl_pin_headers:Pin_Header_Straight_Round_1x01, symbol Connector_Generic:Conn_01x01
- removed P8: COPI, pkl_pin_headers:Pin_Header_Straight_Round_1x01, symbol Connector_Generic:Conn_01x01
- removed P9: IO3, pkl_pads:PAD_SMD_R_1x1, symbol Connector_Generic:Conn_01x01
- removed R1: 1M, pkl_dipol:R_0402, symbol pkl_device:pkl_R_Small
- removed R10, R9: 22E, pkl_dipol:R_0402, symbol pkl_device:pkl_R_Small
- removed R11, R12, R13: 2k2, pkl_dipol:R_0402, symbol pkl_device:pkl_R_Small
- removed R14: 100E, pkl_dipol:R_0402, symbol pkl_device:pkl_R_Small
- removed R2, R6, R8: 10k, pkl_dipol:R_0402, symbol pkl_device:pkl_R_Small
- removed R3, R4: 5k1, pkl_dipol:R_0402, symbol pkl_device:pkl_R_Small
- removed R5: 10k, pkl_dipol:R_Array_Convex_4x0402, symbol pkl_device:pkl_R4_Small
- removed R7: 1k5, pkl_dipol:R_0402, symbol pkl_device:pkl_R_Small
- removed SW1: TACT, pkl_buttons_switches:SW_SPST_3x4x2.5, symbol pkl_misc:TACT
- removed TP1: CC1, pkl_misc:TestPoint_Pad_D0.75mm, symbol Connector:TestPoint_Small
- removed TP2: CC2, pkl_misc:TestPoint_Pad_D0.75mm, symbol Connector:TestPoint_Small
- removed TP3: SBU1, pkl_misc:TestPoint_Pad_D0.75mm, symbol Connector:TestPoint_Small
- removed TP4: SBU2, pkl_misc:TestPoint_Pad_D0.75mm, symbol Connector:TestPoint_Small
- removed U1: LY68L6400, Package_SO:SOIC-8_3.9x4.9mm_P1.27mm, symbol pkl_memory:VTI7064
- removed U2: W25Q128JVxxM, Package_SON:WSON-8-1EP_6x5mm_P1.27mm_EP3.4x4.3mm, symbol pkl_memory:W25Q
- removed U3: TLV75533PDRV, Package_SON:WSON-6-1EP_2x2mm_P0.65mm_EP1x1.6mm, symbol Regulator_Linear:TLV75533PDRV
- removed U4: USBLC6-2, pkl_housings_sot:SOT-666, symbol pkl_misc:USBLC6-2
- removed U5: TLV73312PDRV, Package_SON:WSON-6-1EP_2x2mm_P0.65mm_EP1x1.6mm, symbol Regulator_Linear:TLV75512PDRV
- removed U6: ICE40UP5K-SG48, pkl_housings_dfn_qfn:QFN-48-1EP_7x7mm_Pitch0.5mm, symbol pkl_lattice:ICE40UP5K-SG48
- removed X1: 12MHz, pkl_misc:Oscillator_SMD_SCTF_S2DXX-4Pin_2.5x2.0mm, symbol Oscillator:ASE-xxxMHz
Other:
- removed sheet rp2040
- added sheet address (address.kicad_sch)
- added sheet audio (audio.kicad_sch)
- added sheet microcontroller (microcontroller.kicad_sch)
- added sheet prism-0 (prism.kicad_sch)
- added sheet prism-1 (prism.kicad_sch)
- added sheet prism-2 (prism.kicad_sch)
- added sheet prism-3 (prism.kicad_sch)
- added sheet prism-4 (prism.kicad_sch)
- added sheet prism-5 (prism.kicad_sch)
- added sheet prism-6 (prism.kicad_sch)
- sheet power ports: added VBB; removed ENABLE_FAN, ENABLE_VIO, VIO, VM
- note removed: "+"
- note removed: "-"
- note removed: "128M Flash"
- note removed: "1V2 VReg"
- note removed: "3V3 VReg"
- note removed: "64M PSRAM"
- note removed: "Button"
- note removed: "Chip Select"
- note removed: "Clock"
- note removed: "DPair"
- note removed: "Enable Delay ~1 millisecond Should enable after 1V2 rail"
- note removed: "FPGA"
- note removed: "Flash/RAM"
- note removed: "Hold"
- note removed: "JP3: Cut jumper when only programming iCE Connect jumper for programming Flash and for normal operation"
- note removed: "LEDs"
- note removed: "Main In Secondary Out"
- note removed: "Main Out Secondary In"
- note removed: "Power Pins"
- note removed: "QSPI/Programming"
- note removed: "Serial Clock"
- note removed: "USB"
- note removed: "Using same values as STM32F1 spec"
- note removed: "Write Protect"
- note removed: "or less"

Commit message: Initial components
Parts:
- added U2: PCA9685BS, Janelia:QFN-28-1EP_6x6mm_P0.65mm_EP4.25x4.25mm, symbol Janelia:PCA9685BS
Connections:
- net +3.3V: now also U2.25 (VDD)
- net GND: now also U2.1 (A3), U2.11 (VSS), U2.2 (A4), U2.21 (A5), U2.22 (EXTCLK), U2.26 (A0), U2.27 (A1), U2.28 (A2), U2.29 (VSS)
- net SCL: now also U2.23 (SCL)
- net SDA: now also U2.24 (SDA)
- new net PWM_0: U2.3 (LED0)
- new net PWM_1: U2.4 (LED1)
- new net PWM_2: U2.5 (LED2)
- new net PWM_3: U2.6 (LED3)
- new net PWM_4: U2.7 (LED4)
- new net PWM_5: U2.8 (LED5)
- new net ~{ENABLE}: U2.20 (~{OE})
- no-connect marks 0 -> 10
Other:
- removed sheet address
- removed sheet audio
- removed sheet prism-0
- removed sheet prism-1
- removed sheet prism-2
- removed sheet prism-3
- removed sheet prism-4
- removed sheet prism-5
- removed sheet prism-6
- sheet microcontroller ports: added none; removed AUDIO, PRISM_CIPO, PRISM_COPI, PRISM_SCK, ~{ADDRESS_INT}, ~{ADDRESS_RESET}, ~{PRISMS_RESET}, ~{PRISM_CS_0}, ~{PRISM_CS_1}, ~{PRISM_CS_2}, ~{PRISM_CS_3}, ~{PRISM_CS_4}, ~{PRISM_CS_5}, ~{PRISM_CS_6}
- sheet power ports: added +6V; removed VBB
