File: thruster-pcb/thruster-pcb.kicad_sch (KiCad schematic)
At the start: 1 part, among them U2 PCA9685BS

Commit message: Add sheets
Parts:
- removed U2: PCA9685BS, Janelia:QFN-28-1EP_6x6mm_P0.65mm_EP4.25x4.25mm, symbol Janelia:PCA9685BS
Connections:
- no-connect marks 10 -> 0
Other:
- added sheet thrusters (thrusters.kicad_sch)
Changed lines of the file:
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@@
     (company "Mechatronic Magic")
   )
-  (no_connect (at 209.55 90.17))
-  (no_connect (at 209.55 82.55))
-  (no_connect (at 209.55 72.39))
-  (no_connect (at 209.55 77.47))
-  (no_connect (at 209.55 74.93))
-  (no_connect (at 209.55 85.09))
-  (no_connect (at 209.55 92.71))
-  (no_connect (at 209.55 80.01))
-  (no_connect (at 209.55 87.63))
-  (no_connect (at 209.55 95.25))
-  (wire (pts (xy 191.77 46.99) (xy 191.77 49.53))
-    (stroke (width 0) (type default))
-  )
-  (wire (pts (xy 189.23 105.41) (xy 189.23 102.87))
-    (stroke (width 0) (type default))
-  )
-  (wire (pts (xy 171.45 85.09) (xy 173.99 85.09))
-    (stroke (width 0) (type default))
-  )
   (wire (pts (xy 123.19 48.26) (xy 120.65 48.26))
-    (stroke (width 0) (type default))
-  )
-  (wire (pts (xy 171.45 80.01) (xy 173.99 80.01))
-    (stroke (width 0) (type default))
-  )
-  (wire (pts (xy 171.45 57.15) (xy 173.99 57.15))
-    (stroke (width 0) (type default))
-  )
-  (wire (pts (xy 212.09 57.15) (xy 209.55 57.15))
-    (stroke (width 0) (type default))
-  )
-  (wire (pts (xy 212.09 62.23) (xy 209.55 62.23))
     (stroke (width 0) (type default))
   )
@@
     (stroke (width 0) (type default))
   )
-  (wire (pts (xy 212.09 59.69) (xy 209.55 59.69))
-    (stroke (width 0) (type default))
-  )
   (wire (pts (xy 123.19 45.72) (xy 120.65 45.72))
     (stroke (width 0) (type default))
   )
-  (wire (pts (xy 171.45 90.17) (xy 173.99 90.17))
-    (stroke (width 0) (type default))
-  )
   (wire (pts (xy 87.63 68.58) (xy 90.17 68.58))
-    (stroke (width 0) (type default))
-  )
-  (wire (pts (xy 212.09 69.85) (xy 209.55 69.85))
     (stroke (width 0) (type default))
   )
@@
     (stroke (width 0) (type default))
   )
-  (wire (pts (xy 191.77 105.41) (xy 191.77 102.87))
-    (stroke (width 0) (type default))
-  )
-  (wire (pts (xy 171.45 64.77) (xy 173.99 64.77))
-    (stroke (width 0) (type default))
-  )
   (wire (pts (xy 123.19 66.04) (xy 120.65 66.04))
-    (stroke (width 0) (type default))
-  )
-  (wire (pts (xy 212.09 67.31) (xy 209.55 67.31))
     (stroke (width 0) (type default))
   )
@@
     (stroke (width 0) (type default))
   )
-  (wire (pts (xy 171.45 62.23) (xy 173.99 62.23))
-    (stroke (width 0) (type default))
-  )
   (wire (pts (xy 123.19 76.2) (xy 120.65 76.2))
     (stroke (width 0) (type default))
-  )
-  (wire (pts (xy 171.45 87.63) (xy 173.99 87.63))
-    (stroke (width 0) (type default))
-  )
-  (wire (pts (xy 171.45 59.69) (xy 173.99 59.69))
-    (stroke (width 0) (type default))
-  )
-  (wire (pts (xy 171.45 92.71) (xy 173.99 92.71))
-    (stroke (width 0) (type default))
-  )
-  (wire (pts (xy 212.09 64.77) (xy 209.55 64.77))
-    (stroke (width 0) (type default))
-  )
-  (wire (pts (xy 171.45 82.55) (xy 173.99 82.55))
-    (stroke (width 0) (type default))
-  )
-  (label "PWM_1" (at 212.09 59.69 0) (fields_autoplaced)
-    (effects (font (size 1.27 1.27)) (justify left bottom))
   )
   (label "GND" (at 123.19 50.8 0) (fields_autoplaced)
     (effects (font (size 1.27 1.27)) (justify left bottom))
   )
-  (label "GND" (at 171.45 80.01 180) (fields_autoplaced)
-    (effects (font (size 1.27 1.27)) (justify right bottom))
-  )
-  (label "GND" (at 171.45 92.71 180) (fields_autoplaced)
-    (effects (font (size 1.27 1.27)) (justify right bottom))
-  )
-  (label "SDA" (at 171.45 59.69 180) (fields_autoplaced)
-    (effects (font (size 1.27 1.27)) (justify right bottom))
-  )
-  (label "GND" (at 171.45 82.55 180) (fields_autoplaced)
-    (effects (font (size 1.27 1.27)) (justify right bottom))
-  )
   (label "+5V" (at 123.19 48.26 0) (fields_autoplaced)
-    (effects (font (size 1.27 1.27)) (justify left bottom))
-  )
-  (label "PWM_5" (at 212.09 69.85 0) (fields_autoplaced)
     (effects (font (size 1.27 1.27)) (justify left bottom))
   )
@@
     (effects (font (size 1.27 1.27)) (justify right bottom))
   )
-  (label "PWM_4" (at 212.09 67.31 0) (fields_autoplaced)
-    (effects (font (size 1.27 1.27)) (justify left bottom))
-  )
-  (label "GND" (at 189.23 105.41 270) (fields_autoplaced)
-    (effects (font (size 1.27 1.27)) (justify right bottom))
-  )
   (label "SCL" (at 123.19 76.2 0) (fields_autoplaced)
     (effects (font (size 1.27 1.27)) (justify left bottom))
   )
-  (label "GND" (at 191.77 105.41 270) (fields_autoplaced)
-    (effects (font (size 1.27 1.27)) (justify right bottom))
-  )
-  (label "~{ENABLE}" (at 171.45 64.77 180) (fields_autoplaced)
-    (effects (font (size 1.27 1.27)) (justify right bottom))
-  )
   (label "SDA" (at 123.19 73.66 0) (fields_autoplaced)
-    (effects (font (size 1.27 1.27)) (justify left bottom))
-  )
-  (label "PWM_3" (at 212.09 64.77 0) (fields_autoplaced)
-    (effects (font (size 1.27 1.27)) (justify left bottom))
-  )
-  (label "PWM_0" (at 212.09 57.15 0) (fields_autoplaced)
     (effects (font (size 1.27 1.27)) (justify left bottom))
   )
@@
     (effects (font (size 1.27 1.27)) (justify right bottom))
   )
-  (label "SCL" (at 171.45 57.15 180) (fields_autoplaced)
-    (effects (font (size 1.27 1.27)) (justify right bottom))
-  )
   (label "GND" (at 87.63 34.29 180) (fields_autoplaced)
-    (effects (font (size 1.27 1.27)) (justify right bottom))
-  )
-  (label "GND" (at 171.45 85.09 180) (fields_autoplaced)
     (effects (font (size 1.27 1.27)) (justify right bottom))
   )
@@
     (effects (font (size 1.27 1.27)) (justify left bottom))
   )
-  (label "GND" (at 171.45 62.23 180) (fields_autoplaced)
-    (effects (font (size 1.27 1.27)) (justify right bottom))
-  )
-  (label "GND" (at 171.45 87.63 180) (fields_autoplaced)
-    (effects (font (size 1.27 1.27)) (justify right bottom))
-  )
-  (label "GND" (at 171.45 90.17 180) (fields_autoplaced)
-    (effects (font (size 1.27 1.27)) (justify right bottom))
-  )
-  (label "PWM_2" (at 212.09 62.23 0) (fields_autoplaced)
-    (effects (font (size 1.27 1.27)) (justify left bottom))
-  )
   (label "+6V" (at 123.19 45.72 0) (fields_autoplaced)
     (effects (font (size 1.27 1.27)) (justify left bottom))
-  )
-  (label "+3.3V" (at 191.77 46.99 90) (fields_autoplaced)
-    (effects (font (size 1.27 1.27)) (justify left bottom))
-  )
-  (symbol (lib_id "Janelia:PCA9685BS") (at 191.77 74.93 0) (unit 1)
-    (in_bom yes) (on_board yes) (dnp no) (fields_autoplaced)
-    (property "Reference" "U2" (at 193.9641 49.53 0)
-      (effects (font (size 1.27 1.27)) (justify left))
-    )
-    (property "Value" "PCA9685BS" (at 193.9641 52.07 0)
-      (effects (font (size 1.27 1.27)) (justify left))
-    )
-    (property "Footprint" "Janelia:QFN-28-1EP_6x6mm_P0.65mm_EP4.25x4.25mm" (at 192.405 99.695 0)
-      (effects (font (size 1.27 1.27)) (justify left) hide)
-    )
-    (property "Datasheet" "http://www.nxp.com/docs/en/data-sheet/PCA9685.pdf" (at 191.77 36.83 0)
-      (effects (font (size 1.27 1.27)) hide)
-    )
-    (property "Synopsis" "IC LED DRVR LIN PWM 25MA" (at 191.77 74.93 0)
-      (effects (font (size 1.27 1.27)) hide)
-    )
-    (property "Manufacturer" "NXP Semicon" (at 191.77 74.93 0)
-      (effects (font (size 1.27 1.27)) hide)
-    )
-    (property "Manufacturer Part Number" "PCA9685BS,118" (at 191.77 74.93 0)
-      (effects (font (size 1.27 1.27)) hide)
-    )
-    (property "Vendor" "Digi-Key" (at 191.77 74.93 0)
-      (effects (font (size 1.27 1.27)) hide)
-    )
-    (property "Vendor Part Number" "568-5305-2-ND" (at 191.77 74.93 0)
-      (effects (font (size 1.27 1.27)) hide)
-    )
-    (property "LCSC" "C5191634" (at 191.77 74.93 0)
-      (effects (font (size 1.27 1.27)) hide)
-    )
-    (property "Package" "SOT-788-1" (at 191.77 74.93 0)
-      (effects (font (size 1.27 1.27)) hide)
-    )
-    (pin "24")
-    (pin "25")
-    (pin "26")
-    (pin "3")
-    (pin "28")
-    (pin "23")
-    (pin "9")
-    (pin "29")
-    (pin "27")
-    (pin "4")
-    (pin "22")
-    (pin "21")
-    (pin "2")
-    (pin "20")
-    (pin "18")
-    (pin "8")
-    (pin "17")
-    (pin "19")
-    (pin "16")
-    (pin "7")
-    (pin "5")
-    (pin "15")
-    (pin "14")
-    (pin "6")
-    (pin "10")
-    (pin "11")
-    (pin "12")
-    (pin "13")
-    (pin "1")
-    (instances
-      (project "thruster-pcb"
-        (path "/df2b2e89-e055-4140-95de-f1df723db034"
-          (reference "U2") (unit 1)
-        )
-      )
-    )
   )
   (sheet (at 90.17 31.75) (size 30.48 5.08) (fields_autoplaced)
@@
       )
     )
+  )
+  (sheet (at 175.26 39.37) (size 50.8 43.18) (fields_autoplaced)
+    (stroke (width 0.1524) (type solid))
+    (fill (color 0 0 0 0.0000))
+    (property "Sheetname" "thrusters" (at 175.26 38.6584 0)
+      (effects (font (size 1.27 1.27)) (justify left bottom))
+    )
+    (property "Sheetfile" "thrusters.kicad_sch" (at 175.26 83.1346 0)
+      (effects (font (size 1.27 1.27)) (justify left top))
+    )
+    (instances
+      (project "thruster-pcb"
+        (path "/df2b2e89-e055-4140-95de-f1df723db034" (page "5"))
+      )
+    )

Commit message: Initial schematic and layout
Parts:
- added G101: LOGO-10mm, MechatronicMagicLogo:logo-white-fg-black-bg-10mm, symbol MechatronicMagicLogo:mechatronicmagic-logo-10mm
Other:
- sheet thrusters ports: added +3.3V, +5V, +6V, GND, SCL, SDA; removed none
Changed lines of the file:
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@@
   (title_block
     (title "thruster-pcb")
-    (date "2024-10-22")
-    (rev "2.1")
+    (date "2025-02-17")
+    (rev "1.0")
     (company "Mechatronic Magic")
   )
+  (wire (pts (xy 158.75 57.15) (xy 161.29 57.15))
+    (stroke (width 0) (type default))
+  )
   (wire (pts (xy 123.19 48.26) (xy 120.65 48.26))
+    (stroke (width 0) (type default))
+  )
+  (wire (pts (xy 158.75 49.53) (xy 161.29 49.53))
     (stroke (width 0) (type default))
   )
@@
     (stroke (width 0) (type default))
   )
+  (wire (pts (xy 158.75 52.07) (xy 161.29 52.07))
+    (stroke (width 0) (type default))
+  )
   (wire (pts (xy 123.19 50.8) (xy 120.65 50.8))
     (stroke (width 0) (type default))
@@
     (stroke (width 0) (type default))
   )
+  (wire (pts (xy 158.75 62.23) (xy 161.29 62.23))
+    (stroke (width 0) (type default))
+  )
+  (wire (pts (xy 158.75 54.61) (xy 161.29 54.61))
+    (stroke (width 0) (type default))
+  )
+  (wire (pts (xy 158.75 64.77) (xy 161.29 64.77))
+    (stroke (width 0) (type default))
+  )
   (label "GND" (at 123.19 50.8 0) (fields_autoplaced)
     (effects (font (size 1.27 1.27)) (justify left bottom))
   )
+  (label "SDA" (at 158.75 62.23 180) (fields_autoplaced)
+    (effects (font (size 1.27 1.27)) (justify right bottom))
+  )
   (label "+5V" (at 123.19 48.26 0) (fields_autoplaced)
     (effects (font (size 1.27 1.27)) (justify left bottom))
+  )
+  (label "+3.3V" (at 158.75 54.61 180) (fields_autoplaced)
+    (effects (font (size 1.27 1.27)) (justify right bottom))
   )
   (label "GND" (at 87.63 68.58 180) (fields_autoplaced)
@@
     (effects (font (size 1.27 1.27)) (justify left bottom))
   )
+  (label "GND" (at 158.75 57.15 180) (fields_autoplaced)
+    (effects (font (size 1.27 1.27)) (justify right bottom))
+  )
   (label "+5V" (at 87.63 66.04 180) (fields_autoplaced)
     (effects (font (size 1.27 1.27)) (justify right bottom))
@@
     (effects (font (size 1.27 1.27)) (justify left bottom))
   )
+  (label "SCL" (at 158.75 64.77 180) (fields_autoplaced)
+    (effects (font (size 1.27 1.27)) (justify right bottom))
+  )
   (label "+6V" (at 123.19 45.72 0) (fields_autoplaced)
     (effects (font (size 1.27 1.27)) (justify left bottom))
+  )
+  (label "+6V" (at 158.75 49.53 180) (fields_autoplaced)
+    (effects (font (size 1.27 1.27)) (justify right bottom))
+  )
+  (label "+5V" (at 158.75 52.07 180) (fields_autoplaced)
+    (effects (font (size 1.27 1.27)) (justify right bottom))
+  )
+  (symbol (lib_id "MechatronicMagicLogo:mechatronicmagic-logo-10mm") (at 162.56 181.61 0) (unit 1)
+    (in_bom no) (on_board yes) (dnp no) (fields_autoplaced)
+    (property "Reference" "G101" (at 162.56 172.2401 0)
+      (effects (font (size 1.27 1.27)) hide)
+    )
+    (property "Value" "LOGO-10mm" (at 162.56 190.9799 0)
+      (effects (font (size 1.27 1.27)) hide)
+    )
+    (property "Footprint" "MechatronicMagicLogo:logo-white-fg-black-bg-10mm" (at 162.56 181.61 0)
+      (effects (font (size 1.27 1.27)) hide)
+    )
+    (property "Datasheet" "" (at 162.56 181.61 0)
+      (effects (font (size 1.27 1.27)) hide)
+    )
+    (property "Sim.Enable" "0" (at 162.56 181.61 0)
+      (effects (font (size 1.27 1.27)) hide)
+    )
+    (instances
+      (project "thruster-pcb"
+        (path "/df2b2e89-e055-4140-95de-f1df723db034"
+          (reference "G101") (unit 1)
+        )
+      )
+    )
   )
   (sheet (at 90.17 31.75) (size 30.48 5.08) (fields_autoplaced)
@@
     )
   )
-  (sheet (at 175.26 39.37) (size 50.8 43.18) (fields_autoplaced)
+  (sheet (at 161.29 46.99) (size 12.7 20.32) (fields_autoplaced)
     (stroke (width 0.1524) (type solid))
     (fill (color 0 0 0 0.0000))
-    (property "Sheetname" "thrusters" (at 175.26 38.6584 0)
+    (property "Sheetname" "thrusters" (at 161.29 46.2784 0)
       (effects (font (size 1.27 1.27)) (justify left bottom))
     )
-    (property "Sheetfile" "thrusters.kicad_sch" (at 175.26 83.1346 0)
+    (property "Sheetfile" "thrusters.kicad_sch" (at 161.29 67.8946 0)
       (effects (font (size 1.27 1.27)) (justify left top))
     )
+    (pin "SCL" output (at 161.29 64.77 180)
+      (effects (font (size 1.27 1.27)) (justify left))
+    )
+    (pin "SDA" bidirectional (at 161.29 62.23 180)
+      (effects (font (size 1.27 1.27)) (justify left))
+    )
+    (pin "+3.3V" passive (at 161.29 54.61 180)
+      (effects (font (size 1.27 1.27)) (justify left))
+    )
+    (pin "GND" passive (at 161.29 57.15 180)
+      (effects (font (size 1.27 1.27)) (justify left))
+    )
+    (pin "+5V" passive (at 161.29 52.07 180)
+      (effects (font (size 1.27 1.27)) (justify left))
+    )
+    (pin "+6V" passive (at 161.29 49.53 180)
+      (effects (font (size 1.27 1.27)) (justify left))
+    )
     (instances
