File: thruster-pcb/assembly.kicad_sch (KiCad schematic)
At the start: 8 parts

Commit message: tmc5160-usb -> thruster-pcb
Other:
- title: tmc5160-usb -> thruster-pcb
Changed lines of the file:
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@@
   (paper "A4")
   (title_block
-    (title "tmc5160-usb")
+    (title "thruster-pcb")
     (date "2024-05-10")
     (rev "1.0")
@@
     (pin "1")
     (instances
-      (project "tmc5160-usb"
+      (project "thruster-pcb"
         (path "/df2b2e89-e055-4140-95de-f1df723db034/0ec4fe58-7f94-4826-b0e2-2bc8f3ffe81e"
           (reference "H201") (unit 1)
@@
     )
     (instances
-      (project "tmc5160-usb"
+      (project "thruster-pcb"
         (path "/df2b2e89-e055-4140-95de-f1df723db034/0ec4fe58-7f94-4826-b0e2-2bc8f3ffe81e"
           (reference "FID202") (unit 1)
@@
     (pin "1")
     (instances
-      (project "tmc5160-usb"
+      (project "thruster-pcb"
         (path "/df2b2e89-e055-4140-95de-f1df723db034/0ec4fe58-7f94-4826-b0e2-2bc8f3ffe81e"
           (reference "H204") (unit 1)
@@
     (pin "1")
     (instances
-      (project "tmc5160-usb"
+      (project "thruster-pcb"
         (path "/df2b2e89-e055-4140-95de-f1df723db034/0ec4fe58-7f94-4826-b0e2-2bc8f3ffe81e"
           (reference "H203") (unit 1)
@@
     )
     (instances
-      (project "tmc5160-usb"
+      (project "thruster-pcb"
         (path "/df2b2e89-e055-4140-95de-f1df723db034/0ec4fe58-7f94-4826-b0e2-2bc8f3ffe81e"
           (reference "FID204") (unit 1)
@@
     )
     (instances
-      (project "tmc5160-usb"
+      (project "thruster-pcb"
         (path "/df2b2e89-e055-4140-95de-f1df723db034/0ec4fe58-7f94-4826-b0e2-2bc8f3ffe81e"
           (reference "FID201") (unit 1)
@@
     (pin "1")
     (instances
-      (project "tmc5160-usb"
+      (project "thruster-pcb"
         (path "/df2b2e89-e055-4140-95de-f1df723db034/0ec4fe58-7f94-4826-b0e2-2bc8f3ffe81e"
           (reference "H202") (unit 1)
@@
     )
     (instances
-      (project "tmc5160-usb"
+      (project "thruster-pcb"
         (path "/df2b2e89-e055-4140-95de-f1df723db034/0ec4fe58-7f94-4826-b0e2-2bc8f3ffe81e"
           (reference "FID203") (unit 1)

Commit message: Add reference files
Other:
- company: Howard Hughes Medical Institute -> Mechatronic Magic
Changed lines of the file:
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@@
   (title_block
     (title "thruster-pcb")
-    (date "2024-05-10")
+    (date "2025-01-04")
     (rev "1.0")
-    (company "Howard Hughes Medical Institute")
+    (company "Mechatronic Magic")
   )
   (wire (pts (xy 149.86 138.43) (xy 149.86 140.97))
