File: thruster-pcb/microcontroller.kicad_sch (KiCad schematic)
At the start: 4 parts

Commit message: Initial components
Parts:
- removed A401: PICO_W5500_EVB, Janelia:Pico-W5500-EVB_Header_Holes, symbol Janelia:PICO-W5500-EVB_HEADER_HOLES
- added FW1: FEATHERWING_nRF52_HEADERS, Janelia:FEATHERWING_HEADERS, symbol Janelia:FEATHERWING_nRF52_HEADERS
Connections:
- net +3.3V: now also FW1.2 (3V3)
- net GND: now also FW1.4 (GND)
- net SCL: now also FW1.18 (GPIOSCL/23)
- net SDA: now also FW1.17 (GPIOSDA/22)
- net VSYS renamed VBUS
- net VBUS: now also FW1.26 (USB/VBUS(4.5-5.2V))
- no-connect marks 15 -> 0

Commit message: Add sheets
Parts:
- renumbered FW1 to FW401
Connections:
- no-connect marks 0 -> 23
Changed lines of the file:
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@@
     (company "Mechatronic Magic")
   )
+  (no_connect (at 106.68 125.73))
+  (no_connect (at 149.86 105.41))
+  (no_connect (at 106.68 123.19))
+  (no_connect (at 106.68 107.95))
+  (no_connect (at 106.68 120.65))
+  (no_connect (at 106.68 97.79))
+  (no_connect (at 106.68 110.49))
+  (no_connect (at 149.86 110.49))
+  (no_connect (at 106.68 113.03))
+  (no_connect (at 106.68 105.41))
+  (no_connect (at 106.68 115.57))
+  (no_connect (at 149.86 115.57))
+  (no_connect (at 149.86 120.65))
+  (no_connect (at 149.86 113.03))
+  (no_connect (at 149.86 123.19))
+  (no_connect (at 106.68 92.71))
+  (no_connect (at 149.86 102.87))
+  (no_connect (at 149.86 118.11))
+  (no_connect (at 106.68 130.81))
+  (no_connect (at 106.68 128.27))
+  (no_connect (at 149.86 125.73))
+  (no_connect (at 106.68 118.11))
+  (no_connect (at 106.68 102.87))
   (wire (pts (xy 207.01 46.99) (xy 207.01 49.53))
     (stroke (width 0) (type default))
@@
   (symbol (lib_id "Janelia:FEATHERWING_nRF52_HEADERS") (at 128.27 111.76 0) (unit 1)
     (in_bom no) (on_board yes) (dnp no) (fields_autoplaced)
-    (property "Reference" "FW1" (at 128.27 82.55 0)
+    (property "Reference" "FW401" (at 128.27 82.55 0)
       (effects (font (size 1.27 1.27)))
     )
@@
       (project "thruster-pcb"
         (path "/df2b2e89-e055-4140-95de-f1df723db034/90ad6836-1738-4b32-a341-0a0b169f4662"
-          (reference "FW1") (unit 1)
-        )
-      )
+          (reference "FW401") (unit 1)
+        )
+      )

Commit message: Initial schematic and layout
Changed lines of the file:
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@@
   (title_block
     (title "thruster-pcb")
-    (date "2024-10-22")
-    (rev "2.1")
+    (date "2025-02-17")
+    (rev "1.0")
     (company "Mechatronic Magic")
   )
@@
   (no_connect (at 106.68 118.11))
   (no_connect (at 106.68 102.87))
-  (wire (pts (xy 207.01 46.99) (xy 207.01 49.53))
-    (stroke (width 0) (type default))
-  )
   (wire (pts (xy 226.06 88.9) (xy 226.06 91.44))
     (stroke (width 0) (type default))
@@
   )
   (wire (pts (xy 58.42 54.61) (xy 60.96 54.61))
-    (stroke (width 0) (type default))
-  )
-  (wire (pts (xy 195.58 46.99) (xy 195.58 49.53))
     (stroke (width 0) (type default))
   )
@@
     (effects (font (size 1.27 1.27)) (justify right bottom))
   )
-  (label "+3.3V" (at 207.01 49.53 270) (fields_autoplaced)
-    (effects (font (size 1.27 1.27)) (justify right bottom))
-  )
   (label "+5V" (at 133.35 58.42 180) (fields_autoplaced)
     (effects (font (size 1.27 1.27)) (justify right bottom))
@@
   (label "+5V" (at 60.96 44.45 0) (fields_autoplaced)
     (effects (font (size 1.27 1.27)) (justify left bottom))
-  )
-  (label "VBUS" (at 195.58 49.53 270) (fields_autoplaced)
-    (effects (font (size 1.27 1.27)) (justify right bottom))
   )
   (label "GND" (at 60.96 49.53 0) (fields_autoplaced)
@@
         )
       )
-    )
-  )
-  (symbol (lib_id "power:PWR_FLAG") (at 195.58 46.99 0) (unit 1)
-    (in_bom yes) (on_board yes) (dnp no)
-    (property "Reference" "#FLG0401" (at 195.58 45.085 0)
-      (effects (font (size 1.27 1.27)) hide)
-    )
-    (property "Value" "PWR_FLAG" (at 195.58 43.18 0)
-      (effects (font (size 1.27 1.27)))
-    )
-    (property "Footprint" "" (at 195.58 46.99 0)
-      (effects (font (size 1.27 1.27)) hide)
-    )
-    (property "Datasheet" "~" (at 195.58 46.99 0)
-      (effects (font (size 1.27 1.27)) hide)
-    )
-    (pin "1")
-    (instances
-      (project "thruster-pcb"
-        (path "/df2b2e89-e055-4140-95de-f1df723db034/90ad6836-1738-4b32-a341-0a0b169f4662"
-          (reference "#FLG0401") (unit 1)
-        )
-      )
-    )
-  )
-  (symbol (lib_id "power:PWR_FLAG") (at 207.01 46.99 0) (unit 1)
-    (in_bom yes) (on_board yes) (dnp no)
-    (property "Reference" "#FLG0402" (at 207.01 45.085 0)
-      (effects (font (size 1.27 1.27)) hide)
-    )
-    (property "Value" "PWR_FLAG" (at 207.01 43.18 0)
-      (effects (font (size 1.27 1.27)))
-    )
-    (property "Footprint" "" (at 207.01 46.99 0)
-      (effects (font (size 1.27 1.27)) hide)
-    )
-    (property "Datasheet" "~" (at 207.01 46.99 0)
-      (effects (font (size 1.27 1.27)) hide)
-    )
-    (pin "1")
-    (instances
-      (project "thruster-pcb"
-        (path "/df2b2e89-e055-4140-95de-f1df723db034/90ad6836-1738-4b32-a341-0a0b169f4662"
-          (reference "#FLG0402") (unit 1)
-        )
-      )

Commit message: Initial layout
Parts:
- added C401: 0.1uF_100V, Janelia:C_0402_1005Metric, symbol Janelia:C_0.1uF_100V_0402
- added SW401: SW_DIP_x01_EM-01KP, Janelia:SW_SPST_EM-01KP, symbol Janelia:SW_DIP_x01_EM-01KP
- added U401: MAX6816, Janelia:SOT192P237X122-4N, symbol Janelia:MAX6816
Connections:
- net +3.3V: now also C401.1, U401.4 (Vcc)
- net GND: now also C401.2, SW401.1, U401.1 (GND)
- net RUN_DEBOUNCED: now reaches FW401.5 (GPIOA0/14)
- net RUN_DEBOUNCED: now also U401.3 (OUT)
- new net RUN: SW401.2, U401.2 (IN)
- no-connect marks 23 -> 22
Changed lines of the file:
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@@
   (title_block
     (title "thruster-pcb")
-    (date "2025-02-17")
+    (date "2025-02-18")
     (rev "1.0")
     (company "Mechatronic Magic")
@@
   (no_connect (at 149.86 125.73))
   (no_connect (at 106.68 118.11))
-  (no_connect (at 106.68 102.87))
   (wire (pts (xy 226.06 88.9) (xy 226.06 91.44))
     (stroke (width 0) (type default))
@@
     (stroke (width 0) (type default))
   )
+  (wire (pts (xy 26.67 134.62) (xy 26.67 137.16))
+    (stroke (width 0) (type default))
+  )
+  (wire (pts (xy 55.88 121.92) (xy 55.88 119.38))
+    (stroke (width 0) (type default))
+  )
   (wire (pts (xy 149.86 130.81) (xy 152.4 130.81))
     (stroke (width 0) (type default))
@@
     (stroke (width 0) (type default))
   )
+  (wire (pts (xy 26.67 124.46) (xy 26.67 121.92))
+    (stroke (width 0) (type default))
+  )
   (wire (pts (xy 106.68 95.25) (xy 104.14 95.25))
     (stroke (width 0) (type default))
   )
+  (wire (pts (xy 55.88 105.41) (xy 55.88 107.95))
+    (stroke (width 0) (type default))
+  )
   (wire (pts (xy 58.42 49.53) (xy 60.96 49.53))
     (stroke (width 0) (type default))
@@
     (stroke (width 0) (type default))
   )
+  (wire (pts (xy 66.04 130.81) (xy 68.58 130.81))
+    (stroke (width 0) (type default))
+  )
   (wire (pts (xy 234.95 88.9) (xy 234.95 91.44))
     (stroke (width 0) (type default))
@@
     (stroke (width 0) (type default))
   )
+  (wire (pts (xy 106.68 102.87) (xy 104.14 102.87))
+    (stroke (width 0) (type default))
+  )
   (wire (pts (xy 135.89 58.42) (xy 133.35 58.42))
     (stroke (width 0) (type default))
@@
     (stroke (width 0) (type default))
   )
+  (wire (pts (xy 55.88 90.17) (xy 55.88 87.63))
+    (stroke (width 0) (type default))
+  )
   (wire (pts (xy 234.95 76.2) (xy 234.95 73.66))
     (stroke (width 0) (type default))
   )
+  (wire (pts (xy 45.72 130.81) (xy 43.18 130.81))
+    (stroke (width 0) (type default))
+  )
+  (wire (pts (xy 55.88 137.16) (xy 55.88 139.7))
+    (stroke (width 0) (type default))
+  )
   (label "+3.3V" (at 60.96 46.99 0) (fields_autoplaced)
     (effects (font (size 1.27 1.27)) (justify left bottom))
@@
     (effects (font (size 1.27 1.27)) (justify right bottom))
   )
+  (label "GND" (at 55.88 107.95 270) (fields_autoplaced)
+    (effects (font (size 1.27 1.27)) (justify right bottom))
+  )
+  (label "+3.3V" (at 55.88 119.38 90) (fields_autoplaced)
+    (effects (font (size 1.27 1.27)) (justify left bottom))
+  )
   (label "+5V" (at 133.35 58.42 180) (fields_autoplaced)
     (effects (font (size 1.27 1.27)) (justify right bottom))
   )
+  (label "GND" (at 26.67 137.16 270) (fields_autoplaced)
+    (effects (font (size 1.27 1.27)) (justify right bottom))
+  )
   (label "+3.3V" (at 226.06 73.66 90) (fields_autoplaced)
     (effects (font (size 1.27 1.27)) (justify left bottom))
@@
     (effects (font (size 1.27 1.27)) (justify right bottom))
   )
+  (label "+3.3V" (at 26.67 121.92 90) (fields_autoplaced)
+    (effects (font (size 1.27 1.27)) (justify left bottom))
+  )
+  (label "RUN" (at 43.18 130.81 180) (fields_autoplaced)
+    (effects (font (size 1.27 1.27)) (justify right bottom))
+  )
   (label "SCL" (at 152.4 128.27 0) (fields_autoplaced)
     (effects (font (size 1.27 1.27)) (justify left bottom))
@@
     (effects (font (size 1.27 1.27)) (justify left bottom))
   )
+  (label "RUN_DEBOUNCED" (at 104.14 102.87 180) (fields_autoplaced)
+    (effects (font (size 1.27 1.27)) (justify right bottom))
+  )
+  (label "RUN" (at 55.88 87.63 90) (fields_autoplaced)
+    (effects (font (size 1.27 1.27)) (justify left bottom))
+  )
   (label "SDA" (at 60.96 54.61 0) (fields_autoplaced)
     (effects (font (size 1.27 1.27)) (justify left bottom))
@@
     (effects (font (size 1.27 1.27)) (justify left bottom))
   )
+  (label "GND" (at 55.88 139.7 270) (fields_autoplaced)
+    (effects (font (size 1.27 1.27)) (justify right bottom))
+  )
   (label "GND" (at 60.96 49.53 0) (fields_autoplaced)
     (effects (font (size 1.27 1.27)) (justify left bottom))
   )
   (label "SCL" (at 60.96 52.07 0) (fields_autoplaced)
+    (effects (font (size 1.27 1.27)) (justify left bottom))
+  )
+  (label "RUN_DEBOUNCED" (at 68.58 130.81 0) (fields_autoplaced)
     (effects (font (size 1.27 1.27)) (justify left bottom))
   )
@@
         (path "/df2b2e89-e055-4140-95de-f1df723db034/90ad6836-1738-4b32-a341-0a0b169f4662"
           (reference "R402") (unit 1)
+        )
+      )
+    )
+  )
+  (symbol (lib_id "Janelia:SW_DIP_x01_EM-01KP") (at 55.88 97.79 90) (unit 1)
+    (in_bom yes) (on_board yes) (dnp no) (fields_autoplaced)
+    (property "Reference" "SW401" (at 59.69 96.52 90)
+      (effects (font (size 1.27 1.27)) (justify right))
+    )
+    (property "Value" "SW_DIP_x01_EM-01KP" (at 59.69 99.06 90)
+      (effects (font (size 1.27 1.27)) (justify right))
+    )
+    (property "Footprint" "Janelia:SW_SPST_EM-01KP" (at 55.88 97.79 0)
+      (effects (font (size 1.27 1.27)) hide)
+    )
+    (property "Datasheet" "~" (at 55.88 97.79 0)
+      (effects (font (size 1.27 1.27)) hide)
+    )
+    (property "Synopsis" "1 Digit SPST 24V 25mA DIP" (at 55.88 97.79 0)
+      (effects (font (size 1.27 1.27)) hide)
+    )
+    (property "Manufacturer" "Korean Hroparts Elec" (at 55.88 97.79 0)
+      (effects (font (size 1.27 1.27)) hide)
+    )
+    (property "Manufacturer Part Number" "EM-01KP" (at 55.88 97.79 0)
+      (effects (font (size 1.27 1.27)) hide)
+    )
+    (property "LCSC" "C129077" (at 55.88 97.79 0)
+      (effects (font (size 1.27 1.27)) hide)
+    )
+    (property "Vendor" "jlcpcb" (at 55.88 97.79 0)
+      (effects (font (size 1.27 1.27)) hide)
+    )
+    (property "Vendor Part Number" "C129077" (at 55.88 97.79 0)
+      (effects (font (size 1.27 1.27)) hide)
+    )
+    (property "Package" "SMD,2.5x6mm" (at 55.88 97.79 0)
+      (effects (font (size 1.27 1.27)) hide)
+    )
+    (pin "1")
+    (pin "2")
+    (instances
+      (project "thruster-pcb"
+        (path "/df2b2e89-e055-4140-95de-f1df723db034/90ad6836-1738-4b32-a341-0a0b169f4662"
+          (reference "SW401") (unit 1)
         )
       )
@@
         )
       )
+    )
+  )
+  (symbol (lib_id "Janelia:C_0.1uF_100V_0402") (at 26.67 129.54 0) (unit 1)
+    (in_bom yes) (on_board yes) (dnp no) (fields_autoplaced)
+    (property "Reference" "C401" (at 30.48 128.905 0)
+      (effects (font (size 1.016 1.016)) (justify left))
+    )
+    (property "Value" "0.1uF_100V" (at 30.48 130.8099 0)
+      (effects (font (size 0.762 0.762)) (justify left))
+    )
+    (property "Footprint" "Janelia:C_0402_1005Metric" (at 27.6352 133.35 0)
+      (effects (font (size 0.762 0.762)) hide)
+    )
+    (property "Datasheet" "" (at 26.67 127 0)
+      (effects (font (size 1.524 1.524)) hide)
+    )
+    (property "Vendor" "Digi-Key" (at 29.21 124.46 0)
+      (effects (font (size 1.524 1.524)) hide)
+    )
+    (property "Vendor Part Number" "490-10458-1-ND" (at 31.75 121.92 0)
+      (effects (font (size 1.524 1.524)) hide)
+    )
+    (property "Manufacturer" "Murata Electronics" (at 26.67 129.54 0)
+      (effects (font (size 1.27 1.27)) hide)
+    )
+    (property "Manufacturer Part Number" "GRM155R62A104KE14D" (at 26.67 129.54 0)
+      (effects (font (size 1.27 1.27)) hide)
+    )
+    (property "Package" "0402" (at 26.67 129.54 0)
+      (effects (font (size 1.27 1.27)) hide)
+    )
+    (property "Synopsis" "CAP CER 0.1UF 100V X5R" (at 34.29 119.38 0)
+      (effects (font (size 1.524 1.524)) hide)
+    )
+    (property "LCSC" "C162178" (at 26.67 129.54 0)
+      (effects (font (size 1.27 1.27)) hide)
+    )
+    (pin "2")
+    (pin "1")
+    (instances
+      (project "thruster-pcb"
+        (path "/df2b2e89-e055-4140-95de-f1df723db034/90ad6836-1738-4b32-a341-0a0b169f4662"
+          (reference "C401") (unit 1)
+        )
+      )
+    )
+  )
+  (symbol (lib_id "Janelia:MAX6816") (at 55.88 129.54 0) (unit 1)
+    (in_bom yes) (on_board yes) (dnp no)
+    (property "Reference" "U401" (at 63.5 135.89 0)
+      (effects (font (size 1.524 1.524)))
+    )
+    (property "Value" "MAX6816" (at 63.5 123.19 0) (do_not_autoplace)
+      (effects (font (size 1.524 1.524)))
+    )
+    (property "Footprint" "Janelia:SOT192P237X122-4N" (at 55.88 148.59 0)
+      (effects (font (size 1.524 1.524)) hide)
+    )
+    (property "Datasheet" "" (at 55.88 129.54 0)
+      (effects (font (size 1.524 1.524)))
+    )
+    (property "Package" "SOT-143" (at 55.88 129.54 0)
+      (effects (font (size 1.524 1.524)) hide)
+    )
+    (property "Manufacturer" "Analog Devices Inc./Maxim Integrated" (at 55.88 129.54 0)
+      (effects (font (size 1.524 1.524)) hide)
+    )
+    (property "Manufacturer Part Number" "MAX6816EUS+T" (at 55.88 129.54 0)
+      (effects (font (size 1.524 1.524)) hide)
+    )
+    (property "Vendor" "Digi-Key" (at 55.88 153.67 0)
+      (effects (font (size 1.524 1.524)) hide)
+    )
+    (property "Vendor Part Number" "MAX6816EUS+TCT-ND" (at 55.88 151.13 0)
+      (effects (font (size 1.524 1.524)) hide)
+    )
+    (property "Sim.Enable" "0" (at 55.88 129.54 0)
+      (effects (font (size 1.27 1.27)) hide)
+    )
+    (property "Synopsis" "IC SWITCH DEBOUNCER" (at 55.88 146.05 0)
+      (effects (font (size 1.524 1.524)) hide)
+    )
+    (property "LCSC" "C41637" (at 55.88 129.54 0)
+      (effects (font (size 1.27 1.27)) hide)
+    )
+    (pin "1")
+    (pin "3")
+    (pin "4")
+    (pin "2")
+    (instances
+      (project "thruster-pcb"
+        (path "/df2b2e89-e055-4140-95de-f1df723db034/90ad6836-1738-4b32-a341-0a0b169f4662"
+          (reference "U401") (unit 1)
+        )
+      )
