File: thruster-pcb/power.kicad_sch (KiCad schematic)
At the start: 6 parts, among them U301 TPSM365R6V5RDNR

Commit message: Initial schematic and layout
Parts:
- added J301: Conn_TERM_HDR_01x03_Pin_3.5mm_Horizontal, Janelia:Connector_Header_1x03_P2.54mm_Horizontal_SMD_284052-E, symbol Janelia:Conn_01x03_P2.54_284052-E
Connections:
- net +6V: now also J301.2 (Pin_2)
- net GND: now also J301.1 (Pin_1)
- no-connect marks 4 -> 5
Changed lines of the file:
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@@
   (title_block
     (title "thruster-pcb")
-    (date "2024-10-22")
-    (rev "2.1")
+    (date "2025-02-17")
+    (rev "1.0")
     (company "Mechatronic Magic")
   )
@@
   (no_connect (at 129.54 130.81))
   (no_connect (at 177.8 113.03))
+  (no_connect (at 140.97 66.04))
   (wire (pts (xy 205.74 116.84) (xy 205.74 114.3))
     (stroke (width 0) (type default))
   )
+  (wire (pts (xy 152.4 46.99) (xy 152.4 49.53))
+    (stroke (width 0) (type default))
+  )
   (wire (pts (xy 129.54 113.03) (xy 127 113.03))
     (stroke (width 0) (type default))
@@
     (stroke (width 0) (type default))
   )
-  (wire (pts (xy 129.54 69.85) (xy 132.08 69.85))
-    (stroke (width 0) (type default))
-  )
-  (wire (pts (xy 129.54 67.31) (xy 132.08 67.31))
+  (wire (pts (xy 140.97 71.12) (xy 138.43 71.12))
+    (stroke (width 0) (type default))
+  )
+  (wire (pts (xy 140.97 68.58) (xy 138.43 68.58))
     (stroke (width 0) (type default))
   )
@@
     (stroke (width 0) (type default))
   )
-  (wire (pts (xy 151.13 46.99) (xy 151.13 49.53))
-    (stroke (width 0) (type default))
-  )
-  (wire (pts (xy 162.56 46.99) (xy 162.56 49.53))
-    (stroke (width 0) (type default))
-  )
   (wire (pts (xy 205.74 127) (xy 205.74 129.54))
     (stroke (width 0) (type default))
@@
     (effects (font (size 1.27 1.27)) (justify left bottom))
   )
-  (label "GND" (at 162.56 49.53 270) (fields_autoplaced)
-    (effects (font (size 1.27 1.27)) (justify right bottom))
-  )
-  (label "GND" (at 132.08 69.85 0) (fields_autoplaced)
-    (effects (font (size 1.27 1.27)) (justify left bottom))
+  (label "GND" (at 138.43 71.12 180) (fields_autoplaced)
+    (effects (font (size 1.27 1.27)) (justify right bottom))
   )
   (label "VDD" (at 127 118.11 180) (fields_autoplaced)
     (effects (font (size 1.27 1.27)) (justify right bottom))
   )
+  (label "+5V" (at 152.4 49.53 270) (fields_autoplaced)
+    (effects (font (size 1.27 1.27)) (justify right bottom))
+  )
   (label "+6V" (at 127 125.73 180) (fields_autoplaced)
     (effects (font (size 1.27 1.27)) (justify right bottom))
   )
-  (label "+6V" (at 132.08 67.31 0) (fields_autoplaced)
-    (effects (font (size 1.27 1.27)) (justify left bottom))
+  (label "+6V" (at 138.43 68.58 180) (fields_autoplaced)
+    (effects (font (size 1.27 1.27)) (justify right bottom))
   )
   (label "GND" (at 193.04 129.54 270) (fields_autoplaced)
@@
   (label "+6V" (at 77.47 114.3 90) (fields_autoplaced)
     (effects (font (size 1.27 1.27)) (justify left bottom))
-  )
-  (label "+5V" (at 151.13 49.53 270) (fields_autoplaced)
-    (effects (font (size 1.27 1.27)) (justify right bottom))
   )
   (label "+6V" (at 127 113.03 180) (fields_autoplaced)
@@
         (path "/df2b2e89-e055-4140-95de-f1df723db034/c1dd8f61-494c-402f-8e59-08309c64fc3f"
           (reference "C303") (unit 1)
-        )
-      )
-    )
-  )
-  (symbol (lib_id "power:PWR_FLAG") (at 162.56 46.99 0) (unit 1)
-    (in_bom yes) (on_board yes) (dnp no)
-    (property "Reference" "#FLG0303" (at 162.56 45.085 0)
-      (effects (font (size 1.27 1.27)) hide)
-    )
-    (property "Value" "PWR_FLAG" (at 162.56 43.18 0)
-      (effects (font (size 1.27 1.27)))
-    )
-    (property "Footprint" "" (at 162.56 46.99 0)
-      (effects (font (size 1.27 1.27)) hide)
-    )
-    (property "Datasheet" "~" (at 162.56 46.99 0)
-      (effects (font (size 1.27 1.27)) hide)
-    )
-    (pin "1")
-    (instances
-      (project "thruster-pcb"
-        (path "/df2b2e89-e055-4140-95de-f1df723db034/c1dd8f61-494c-402f-8e59-08309c64fc3f"
-          (reference "#FLG0303") (unit 1)
         )
       )
@@
     )
   )
-  (symbol (lib_id "power:PWR_FLAG") (at 151.13 46.99 0) (unit 1)
-    (in_bom yes) (on_board yes) (dnp no)
-    (property "Reference" "#FLG0302" (at 151.13 45.085 0)
-      (effects (font (size 1.27 1.27)) hide)
-    )
-    (property "Value" "PWR_FLAG" (at 151.13 43.18 0)
-      (effects (font (size 1.27 1.27)))
-    )
-    (property "Footprint" "" (at 151.13 46.99 0)
-      (effects (font (size 1.27 1.27)) hide)
-    )
-    (property "Datasheet" "~" (at 151.13 46.99 0)
-      (effects (font (size 1.27 1.27)) hide)
-    )
-    (pin "1")
-    (instances
-      (project "thruster-pcb"
-        (path "/df2b2e89-e055-4140-95de-f1df723db034/c1dd8f61-494c-402f-8e59-08309c64fc3f"
-          (reference "#FLG0302") (unit 1)
-        )
-      )
-    )
-  )
   (symbol (lib_id "Janelia:C_47uF_10V_0805") (at 205.74 121.92 0) (unit 1)
     (in_bom yes) (on_board yes) (dnp no)
@@
         )
       )
+    )
+  )
+  (symbol (lib_id "Janelia:Conn_01x03_P2.54_284052-E") (at 146.05 68.58 180) (unit 1)
+    (in_bom yes) (on_board yes) (dnp no) (fields_autoplaced)
+    (property "Reference" "J301" (at 147.32 68.58 0)
+      (effects (font (size 1.27 1.27)) (justify right))
+    )
+    (property "Value" "Conn_TERM_HDR_01x03_Pin_3.5mm_Horizontal" (at 146.05 55.88 0)
+      (effects (font (size 1.27 1.27)) hide)
+    )
+    (property "Footprint" "Janelia:Connector_Header_1x03_P2.54mm_Horizontal_SMD_284052-E" (at 146.05 104.14 0)
+      (effects (font (size 1.27 1.27)) hide)
+    )
+    (property "Datasheet" "" (at 146.05 88.9 0)
+      (effects (font (size 1.27 1.27)) hide)
+    )
+    (property "Manufacturer" "TE Connectivity" (at 146.05 101.6 0)
+      (effects (font (size 1.27 1.27)) hide)
+    )
+    (property "Manufacturer Part Number" "284052-E" (at 146.05 96.52 0)
+      (effects (font (size 1.27 1.27)) hide)
+    )
+    (property "Synopsis" "MAXIBR M 03POS RA A SMT BK" (at 146.05 93.98 0)
+      (effects (font (size 1.27 1.27)) hide)
+    )
+    (property "Vendor" "Digi-Key" (at 146.05 99.06 0)
+      (effects (font (size 1.27 1.27)) hide)
+    )
+    (property "Vendor Part Number" "2684-284052-ETR-ND" (at 146.05 91.44 0)
+      (effects (font (size 1.27 1.27)) hide)
+    )
+    (property "Sim.Enable" "0" (at 146.05 68.58 0)
+      (effects (font (size 1.27 1.27)) hide)
+    )
+    (property "LCSC" "C17355078" (at 146.05 68.58 0)
+      (effects (font (size 1.27 1.27)) hide)
+    )
+    (pin "1")
+    (pin "2")
+    (pin "3")
+    (instances
+      (project "thruster-pcb"
+        (path "/df2b2e89-e055-4140-95de-f1df723db034/c1dd8f61-494c-402f-8e59-08309c64fc3f"
+          (reference "J301") (unit 1)
+        )
+      )
+    )
+  )
+  (symbol (lib_id "power:PWR_FLAG") (at 152.4 46.99 0) (unit 1)
+    (in_bom yes) (on_board yes) (dnp no)
+    (property "Reference" "#FLG0302" (at 152.4 45.085 0)
+      (effects (font (size 1.27 1.27)) hide)
+    )
+    (property "Value" "PWR_FLAG" (at 152.4 43.18 0)
+      (effects (font (size 1.27 1.27)))
+    )
+    (property "Footprint" "" (at 152.4 46.99 0)
+      (effects (font (size 1.27 1.27)) hide)
+    )
+    (property "Datasheet" "~" (at 152.4 46.99 0)
+      (effects (font (size 1.27 1.27)) hide)
+    )
+    (pin "1")
+    (instances
+      (project "thruster-pcb"
+        (path "/df2b2e89-e055-4140-95de-f1df723db034/c1dd8f61-494c-402f-8e59-08309c64fc3f"
+          (reference "#FLG0302") (unit 1)
+        )
+      )
