File: thruster-pcb/thrusters.kicad_sch (KiCad schematic)
At the start: 6 parts, among them U501 PCA9685BS, U502 LevelTranslator_TXS0108EPW

Commit message: Initial schematic and layout
Parts:
- added C505, C506, C507, C508, C509: 47uF_10V, Janelia:C_0805_2012Metric, symbol Janelia:C_47uF_10V_0805
- added J501, J502, J503, J504, J505, J506: Conn_TERM_HDR_01x03_Pin_3.5mm_Horizontal, Janelia:Connector_Header_1x03_P2.54mm_Horizontal_SMD_284052-E, symbol Janelia:Conn_01x03_P2.54_284052-E
Connections:
- net +6V: now also C505.1, C506.1, C507.1, C508.1, C509.1, J501.2 (Pin_2), J502.2 (Pin_2), J503.2 (Pin_2), J504.2 (Pin_2), J505.2 (Pin_2), J506.2 (Pin_2)
- net GND: now also C505.2, C506.2, C507.2, C508.2, C509.2, J501.1 (Pin_1), J502.1 (Pin_1), J503.1 (Pin_1), J504.1 (Pin_1), J505.1 (Pin_1), J506.1 (Pin_1)
- net SIG_0: now also J501.3 (Pin_3)
- net SIG_1: now also J502.3 (Pin_3)
- net SIG_2: now also J503.3 (Pin_3)
- net SIG_3: now also J504.3 (Pin_3)
- net SIG_4: now also J505.3 (Pin_3)
- net SIG_5: now also J506.3 (Pin_3)
Other:
- company: (none) -> Mechatronic Magic
- title: (none) -> thruster-pcb
- moved on the sheet: C501, C502, C503, C504, U501, U502
